Commit message: fix: Set camera d435i inclinaison to "0 0 0"

File: src/_gr/Turtlebot3/projects/turtlebot3_descriptions/urdf/turtlebot3_burger_d435i.urdf (robot description, URDF)
Before this commit: robot turtlebot3_burger, 11 links, 10 joints
Joints:
- joint joint_d435i_camera: origin xyz=0.05 0.0 0.12 rpy=0.0 -0.26 0.0 -> xyz=0.05 0.0 0.12 rpy=0.0 0.0 0.0
